Commit message: u

File: xacro/skidbot.xacro (robot description, xacro)
@@ -6,7 +6,7 @@
 <!-- *********************************************************************************************************************************  -->
 <!-- ****************************************************** Parameters ***************************************************************  -->
-  <xacro:property name="mesh_path"      value="package://robot_gazebo/meshes/skidbot/"/>
+  <xacro:property name="mesh_path"      value="package://skidbot/meshes/skidbot/"/>
   <xacro:property name="name_space"     value="skidbot"  />
-  <xacro:property name="prefix"         value=""  />
+  <xacro:property name="prefix"         value=""         />
   <xacro:property name="base_mass"      value="15.0"     /> <!-- arbitrary mass value -->
   <xacro:property name="base_width"     value="0.20"     />
@@ -31,6 +31,6 @@
   <xacro:property name="hokuyo_z"       value="${(hokuyo_height+base_height)/2}" />
 <!-- ****************************************************** Includes *****************************************************************  -->
-  <xacro:include filename="$(find robot_gazebo)/xacro/common_rviz_materials.xacro" />   <!-- RVIZ Colors                                -->
-  <xacro:include filename="$(find robot_gazebo)/gazebo/gz_skidbot.xacro" />             <!-- Gazebo                                     -->
+  <xacro:include filename="$(find skidbot)/xacro/common_rviz_materials.xacro" />   <!-- RVIZ Colors                                     -->
+  <xacro:include filename="$(find skidbot)/gazebo/gz_skidbot.xacro" />             <!-- Gazebo                                          -->
 <!-- ****************************************************** Base Footprint ***********************************************************  -->
   <link name="${prefix}footprint"></link>

Commit message: u

File: xacro/skidbot.xacro (robot description, xacro)
@@ -158,5 +158,5 @@
       <origin xyz="0 0 0" rpy="0 0 0" />
       <geometry>
-        <mesh filename="${mesh_path}hokuyo.dae"/> <!--  <box size="${hokuyo_length} ${hokuyo_width} ${hokuyo_height}"/> -->
+        <box size="${hokuyo_length} ${hokuyo_width} ${hokuyo_height}"/>
       </geometry>
     </collision>
